File: covert2npnGNDPLANES.brd (EAGLE design)
At the start: 50.8 x 33.5 mm, 55 parts, among them J1 B2B-PH-K-S(LF)(SN), U1 STM32G081RBT6, U2 MMBT4401-7-F

Commit message: some more fixes
Parts:
- removed R3: 1k, standardparts:0805
- removed R4: 10k, standardparts:0805
- added C2: 1uF, standardparts:0805
- added C6: 4.7uF, standardparts:0805
- added JP30, JP33: (no value), pinhead:1X01
- 3.3V_REG: value LM1117MPX-3.3/NOPB -> TPS7A0533PDBVR; device LM1117MPX-3.3_NOPB (1):VREG_LM1117MPX-3.3/NOPB -> TPS7A0533PDBVR:SOT95P280X145-5N
- R5, R6: value 1k -> 1.5k
- moved 3.3V_REG 6.27 mm to (41.4, 18.3), turned to 270 degrees
- moved U2 2.41 mm to (14.5, 14.5)
- moved D2 2.03 mm to (33.5, 24.1)
- moved R5 2.03 mm to (35.3, 24.1)
- moved R1 2.03 mm to (21.3, 4.06)
- moved GND 1.55 mm to (43.4, 30.2)
- moved D3 1.52 mm to (23.6, 4.06)
- moved JP2 1.27 mm to (2.54, 6.10)
- moved JP4 1.27 mm to (2.54, 3.56)
- moved D4 1.27 mm to (25.7, 4.06)
- moved JP1 1.27 mm to (2.54, 11.2)
- moved JP3 1.27 mm to (2.54, 8.64)
- moved D1 1.02 mm to (41.7, 24.1)
- moved R6 1.02 mm to (43.4, 24.1)
- moved R7 0.76 mm to (27.9, 4.06)
Connections:
- removed net N$2: LIPO_CHARGER.4, R3.1
- removed net N$3: LIPO_CHARGER.9, R4.2
- net 5VUSB: now also JP30.1; no longer R4.1
- net GND: now also 3.3V_REG.2, C2.1, C6.1, JP33.1, LIPO_CHARGER.11; no longer 3.3V_REG.1, R3.2
- net VCC_1: now also 3.3V_REG.1, C2.2
- net VCC_2_NET: now also 3.3V_REG.5, C6.2; no longer 3.3V_REG.2, 3.3V_REG.4
Routing:
- net VCC_1: track 104.5 -> 86.6 mm
- net N$3: track 6.63 -> 0.00 mm, vias 2 -> 0
- net GND: track 15.4 -> 21.8 mm, vias 20 -> 21
- net N$2: track 4.28 -> 0.00 mm
- net V_VIB_NEG: track 10.6 -> 13.2 mm
- net N$8: track 1.87 -> 3.57 mm
- net SWDCLK: track 21.1 -> 19.8 mm
- net N$7: track 4.16 -> 2.93 mm
- net VCC_2_NET: track 65.0 -> 63.9 mm
- net 5VUSB: track 28.3 -> 27.2 mm
- net N$11: track 4.93 -> 5.68 mm
- net GPIO_OUTPUT1: track 3.82 -> 4.45 mm
- net SWDIO: track 17.2 -> 16.7 mm
- net N$9: track 1.83 -> 2.34 mm
- net N$4: track 1.83 -> 2.34 mm

Commit message: clean up
Parts:
- removed JP25: (no value), pinhead:1X01
- moved C6 0.51 mm to (40.9, 14.5)
- moved 3.3V_REG 0.51 mm to (41.4, 17.8)
Connections:
- net VCC_1 renamed VBAT
- removed net SHIELD: MICRO_USB.SH1, MICRO_USB.SH2, MICRO_USB.SH3, MICRO_USB.SH4, MICRO_USB.SH5, MICRO_USB.SH6, MICRO_USB.SH7, MICRO_USB.SH8
- removed net VCC_2_NET: 3.3V_REG.5, C3.2, C4.2, C6.2, JP16.1, JP25.1, JP4.1, U1.6, U1.8
- new net 3V3: 3.3V_REG.5, C3.2, C4.2, C6.2, JP16.1, JP4.1, U1.6, U1.8
Routing:
- net VCC_2_NET: track 63.9 -> 0.00 mm
- net 3V3: track 0.00 -> 61.6 mm
- net GND: track 21.8 -> 18.5 mm, vias 21 -> 22
- net VBAT: track 86.6 -> 87.7 mm
