File: covert2npnGNDPLANES.sch (EAGLE design)
At the start: 55 parts, among them J1 B2B-PH-K-S(LF)(SN), U1 STM32G081RBT6, U2 MMBT4401-7-F

Commit message: some more fixes
Parts:
- removed R3: 1k, standardparts:RESISTOR.0805
- removed R4: 10k, standardparts:RESISTOR.0805
- added C2: 1uF, standardparts:CAPACITOR.0805
- added C6: 4.7uF, standardparts:CAPACITOR.0805
- added JP30, JP33: (no value), pinhead:PINHD-1X1
- 3.3V_REG: value LM1117MPX-3.3/NOPB -> TPS7A0533PDBVR; device LM1117MPX-3.3_NOPB (1):LM1117MPX-3.3/NOPB -> TPS7A0533PDBVR:TPS7A0533PDBVR
- R5, R6: value 1k -> 1.5k
Connections:
- removed net N$2: LIPO_CHARGER.PRETERM, R3.1
- removed net N$3: LIPO_CHARGER.TS, R4.2
- net 5VUSB: now also JP30.1; no longer R4.1
- net GND: now also C2.1, C6.1, JP33.1, LIPO_CHARGER.EP; no longer R3.2
- net VCC_1: now also 3.3V_REG.EN, 3.3V_REG.IN, C2.2; no longer 3.3V_REG.VIN
- net VCC_2_NET: now also 3.3V_REG.OUT, C6.2; no longer 3.3V_REG.VOUT_2, 3.3V_REG.VOUT_4
Other:
- moved on the sheet: 3.3V_REG

Commit message: clean up
Parts:
- removed JP25: (no value), pinhead:PINHD-1X1
Connections:
- net VCC_1 renamed VBAT
- removed net SHIELD: MICRO_USB.SHIELD
- removed net VCC_2_NET: 3.3V_REG.OUT, C3.2, C4.2, C6.2, JP16.1, JP25.1, JP4.1, U1.VBAT, U1.VDD
- new net 3V3: 3.3V_REG.OUT, C3.2, C4.2, C6.2, JP16.1, JP4.1, U1.VBAT, U1.VDD
