File: covert2temprouted.brd (EAGLE design)
At the start: 50.8 x 33.5 mm, 44 parts, among them J1 B2B-PH-K-S(LF)(SN), U1 STM32G081RBT6

Commit message: clean up
Parts:
- added JP21, JP22, JP23, JP24, JP25, JP26, JP27, JP28, JP29: (no value), pinhead:1X01
- R1, R7: value 1k -> 500
- moved JP18 31.8 mm to (48.0, 2.79)
- moved JP17 23.9 mm to (42.7, 2.79)
- moved JP20 4.93 mm to (37.6, 2.79)
- moved JP19 2.50 mm to (32.5, 2.79)
- moved D3 1.55 mm to (25.1, 4.06)
- moved D4 1.55 mm to (26.9, 4.06)
- moved R7 1.55 mm to (28.7, 4.06)
- moved R1 1.55 mm to (23.4, 4.06)
Connections:
- net GND: now also JP23.1, JP26.1, JP27.1, JP28.1, JP29.1
- net GPIO_INPUT1: now also U1.63; no longer U1.57
- net GPIO_INPUT2: now also U1.64; no longer U1.56
- net RESET: now also JP24.1
- net VCC_1: now also JP21.1
- net VCC_2_NET: now also JP25.1
- net V_VIB_NEG: now also JP22.1
Routing:
- net VCC_2_NET: track 21.3 -> 59.1 mm
- net VCC_1: track 79.8 -> 104.7 mm, vias 1 -> 0
- net GPIO_INPUT2: track 11.9 -> 23.0 mm
- net GPIO_INPUT1: track 10.4 -> 18.4 mm
- net RESET: track 0.00 -> 7.36 mm
- net GPIO_OUTPUT4: track 8.86 -> 14.1 mm
- net GPIO_OUTPUT3: track 7.72 -> 10.1 mm
- net GPIO_OUTPUT1: track 4.70 -> 3.82 mm
- net V_VIB_NEG: track 11.2 -> 11.8 mm, vias 1 -> 0
